File: piezo-jfet.kicad_pcb (KiCad board)
At the start: 2 copper layers, 34 x 68 mm, 24 parts, among them J1 XLR3, J2 Conn_01x01_Female, J3 Conn_01x01_Female, J4 Conn_01x01_Female, J5 Conn_01x01_Female, Q1 J105, Q2 LSK389B, X1 XTAL, X2 XTAL

Commit message: Add files via upload
Updated files.
Parts:
- removed R6: 150, Resistor_THT:R_Axial_DIN0204_L3.6mm_D1.6mm_P5.08mm_Horizontal
- added J6: Conn_01x01_Female, MountingHole:MountingHole_2.2mm_M2_DIN965_Pad, F.Cu at (69.0, 109.0)
- added R5: 150, Resistor_THT:R_Axial_DIN0204_L3.6mm_D1.6mm_P5.08mm_Horizontal, F.Cu at (77.5, 72.5)
Routing:
- net Net-(J1-Pad3): track 35.0 -> 36.5 mm
- net Net-(C2-Pad1): track 11.4 -> 9.92 mm

Commit message: updated files
Parts:
- removed X1, X2: XTAL, Connector_PinSocket_2.54mm:PinSocket_1x02_P2.54mm_Vertical
- added J7: Conn_01x01_Female, MountingHole:MountingHole_2.2mm_M2_DIN965_Pad, F.Cu at (66.5, 96.5)
- added J8: Conn_01x01_Female, MountingHole:MountingHole_2.2mm_M2_DIN965_Pad, F.Cu at (71.5, 96.5)
- added J9: Conn_01x01_Female, MountingHole:MountingHole_2.2mm_M2_DIN965_Pad, F.Cu at (78.0, 96.5)
- moved J6 14.8 mm to (61.0, 96.5)
- moved C1 14.0 mm to (57.0, 77.5)
- moved C2 14.0 mm to (62.5, 58.5)
- moved C3 14.0 mm to (81.0, 80.0)
- moved Q1 14.0 mm to (67.5, 86.5)
- moved Q2 14.0 mm to (69.0, 70.0)
- moved R1 14.0 mm to (57.0, 68.1)
- moved R10 14.0 mm to (77.0, 81.0)
- moved R12 14.0 mm to (69.0, 81.0)
- moved R2 14.0 mm to (61.0, 81.0)
- moved R3 14.0 mm to (61.0, 68.1)
- moved R4 14.0 mm to (65.0, 81.0)
- moved R5 14.0 mm to (77.5, 58.5)
- moved R7 14.0 mm to (77.5, 68.0)
- moved R8 14.0 mm to (73.0, 81.0)
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Connections:
- J6 pad 1: GND -> Net-(C1-Pad2)
Routing:
- net Net-(J1-Pad3): track 36.5 -> 20.6 mm
- net Net-(C2-Pad2): track 36.0 -> 22.0 mm
- net Net-(C1-Pad2): track 17.9 -> 18.4 mm
Other:
- board text added: "Use shielded cable, with 4 leads. Connect outer cable shield to metal box."

Commit message: Add files via upload
Parts:
- added REF**: OSHW-Symbol_6.7x6mm_SilkScreen, Symbol:OSHW-Symbol_6.7x6mm_SilkScreen, F.Cu at (55.5, 87.0)
- Q1: value J105 -> LSK170B
- Q2: footprint SO-239:TO-71-6 -> tastatur:TO-71-6
Other:
- board text added: "+"
- board text added: "1"
- board text added: "2"
- board text added: "3"
- board text added: "Amplifier for piezoelectric crystals, +48 V phantom power."
- board text added: "Licensed under Creative Commons Attribution 4.0 International"

Commit message: Add files via upload
Parts:
- removed J7: Conn_01x01_Female, MountingHole:MountingHole_2.2mm_M2_DIN965_Pad
- removed REF**: OSHW-Symbol_6.7x6mm_SilkScreen, Symbol:OSHW-Symbol_6.7x6mm_SilkScreen
- R12: value 270 -> 40
- moved J8 2.50 mm to (69.0, 96.5)

Commit message: Add files via upload
Parts:
- added J10: Conn_01x01_Female, MountingHole:MountingHole_2.2mm_M2_DIN965_Pad, F.Cu at (74.9, 47.7)
- added J7: Conn_01x01_Female, MountingHole:MountingHole_2.2mm_M2_DIN965_Pad, F.Cu at (69.5, 47.7)
- J1: value XLR3 -> Conn_01x01_Female; footprint Connector_PinSocket_2.54mm:PinSocket_1x03_P2.54mm_Vertical -> MountingHole:MountingHole_2.2mm_M2_DIN965_Pad
- moved J1 2.26 mm to (64.2, 47.7), turned to 0 degrees
Connections:
- C2 pad 2: Net-(C2-Pad2) -> /2
- J1 pad 1: GND -> /2
- R1 pad 2: Net-(C2-Pad2) -> /2
- R3 pad 2: Net-(C2-Pad2) -> /2
- R5 pad 1: Net-(J1-Pad3) -> /3
- R7 pad 2: Net-(J1-Pad3) -> /3
- R9 pad 2: Net-(J1-Pad3) -> /3
Routing:
- net /3: track 0.00 -> 22.7 mm
- net /2: track 0.00 -> 22.4 mm
- net Net-(C2-Pad2): track 22.0 -> 0.00 mm
- net Net-(J1-Pad3): track 20.6 -> 0.00 mm
Other:
- board text added: "GND"
- board text added: "Use shielded cable, with 3 leads. Connect outer cable shield to metal box."
- board text removed: "Use shielded cable, with 4 leads. Connect outer cable shield to metal box."
