File: piezo-jfet.sch (KiCad schematic (older format))
At the start: 24 parts, among them J1 XLR3, J2 Conn_01x01_Female, J3 Conn_01x01_Female, J4 Conn_01x01_Female, J5 Conn_01x01_Female, Q1 J105, Q2 LSK389B, X1 XTAL, X2 XTAL

Commit message: Add files via upload
Updated files.
Parts:
- removed R6: 150, Resistor_THT:R_Axial_DIN0204_L3.6mm_D1.6mm_P5.08mm_Horizontal, symbol Device:R
- added J6: Conn_01x01_Female, MountingHole:MountingHole_2.2mm_M2_DIN965_Pad, symbol Connector:Conn_01x01_Female
- added R5: 150, Resistor_THT:R_Axial_DIN0204_L3.6mm_D1.6mm_P5.08mm_Horizontal, symbol Device:R
Connections:
- net GND: now also J6.1 (Pin_1)
- net at C2.1: now also R5.2
- net at J1.3, R7.2, R9.2: now also R5.1

Commit message: updated files
Parts:
- removed X1, X2: XTAL, Connector_PinSocket_2.54mm:PinSocket_1x02_P2.54mm_Vertical, symbol piezo-jfet-rescue:XTAL-Keyboard
- added J7, J8, J9: Conn_01x01_Female, MountingHole:MountingHole_2.2mm_M2_DIN965_Pad, symbol Connector:Conn_01x01_Female
Connections:
- net GND: now also J7.1 (Pin_1), J8.1 (Pin_1); no longer J6.1 (Pin_1)
- net at C1.2, D1.2 (A): now also J6.1 (Pin_1)
- net at C3.1, D2.2 (A): now also J9.1 (Pin_1)
Other:
- note added: "Connect outer cable shield and plug shield to metal box."
- note added: "This line represent the outside of a metal box."
- note added: "Use shielded cable, with 4 leads.\nConnect outer cable shield to metal box."
- moved on the sheet: C1, C2, C3, D1, D2, J1, J2, J3, J4, J5, Q1, Q2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

Commit message: Add files via upload
Parts:
- Q1: value J105 -> LSK170B
- Q2: footprint SO-239:TO-71-6 -> tastatur:TO-71-6
Other:
- note added: "+"
- note added: "2x 1N5230B-TR can be used."
- note added: "All resistors and caps must be audio grade."
- note added: "All resistors, FETs and capacitators are THT.\nUse film resistors and X7R caps!"
- note added: "All shield connections must be short as possible."
- note added: "For connection to the piezo crystals:\nUse shielded cable, with 4 leads.\nConnect outer cable shield to metal box. \nOuter end of cable shield may be connected to the outer box \nthat houses the crystals if that is used. If not, leave unconnected."
- note added: "Idss: 4.25 mA\n\n\n"
- note removed: "Idss: 4.25 mA\nvds(v): 10 v\nvgs: 0.2 \nvds(v): 10 V\nV GS(OFF): 0.4 V\n"
- note removed: "Use shielded cable, with 4 leads.\nConnect outer cable shield to metal box."
- moved on the sheet: C1, C2, C3, D1, D2, J2, J3, J4, J5, J6, J7, J8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

Commit message: Add files via upload
Parts:
- removed J7: Conn_01x01_Female, MountingHole:MountingHole_2.2mm_M2_DIN965_Pad, symbol Connector:Conn_01x01_Female
- R12: value 270 -> 40
Other:
- note added: "All resistors, FETs and capacitators are THT.\nUse high tolerance film resistors and X7R caps!"
- note added: "For connection to the piezo crystals:\nUse shielded cable, with 3 leads.\nConnect outer cable shield to metal box. \nOuter end of cable shield may be connected to the outer box \nthat houses the crystals if that is used. If not, leave unconnected."
- note removed: "All resistors, FETs and capacitators are THT.\nUse film resistors and X7R caps!"
- note removed: "For connection to the piezo crystals:\nUse shielded cable, with 4 leads.\nConnect outer cable shield to metal box. \nOuter end of cable shield may be connected to the outer box \nthat houses the crystals if that is used. If not, leave unconnected."
- moved on the sheet: J6, J8, J9
Changed lines of the file:
@@
 $EndComp
 Wire Wire Line
-	1450 5850 1450 5450
-Connection ~ 1450 5450
-Wire Wire Line
-	2650 5950 2400 5950
-Wire Wire Line
-	2400 5950 2400 5850
-Connection ~ 2400 5850
-Wire Wire Line
-	2400 5850 2050 5850
+	1900 5850 1900 5450
 $Comp
 L power:GND #PWR03
 U 1 1 609E54F5
-P 2650 5950
-F 0 "#PWR03" H 2650 5700 50  0001 C CNN
-F 1 "GND" H 2655 5777 50  0000 C CNN
-F 2 "" H 2650 5950 50  0001 C CNN
-F 3 "" H 2650 5950 50  0001 C CNN
-	1    2650 5950
-	1    0    0    -1
+P 2800 5750
+F 0 "#PWR03" H 2800 5500 50  0001 C CNN
+F 1 "GND" H 2805 5577 50  0000 C CNN
+F 2 "" H 2800 5750 50  0001 C CNN
+F 3 "" H 2800 5750 50  0001 C CNN
+	1    2800 5750
+	0    -1   -1   0
 $EndComp
 $Comp
@@
 	3000 5450 2450 5450
 Wire Wire Line
-	2150 5450 1450 5450
+	2150 5450 1900 5450
 $Comp
 L Device:R R3
@@
 	3050 5150 4150 5150
 Wire Wire Line
-	1100 5450 1450 5450
-Wire Wire Line
 	2000 1900 2100 1900
 Wire Wire Line
@@
 P 2350 5000
 F 0 "R12" H 2420 5046 50  0000 L CNN
-F 1 "270" H 2420 4955 50  0000 L CNN
+F 1 "40" H 2420 4955 50  0000 L CNN
 F 2 "Resistor_THT:R_Axial_DIN0204_L3.6mm_D1.6mm_P5.08mm_Horizontal" V 2280 5000 50  0001 C CNN
 F 3 "~" H 2350 5000 50  0001 C CNN
@@
 	2050 5150 2350 5150
 Wire Wire Line
-	3850 5450 3850 5850
-Wire Wire Line
-	3800 5850 3850 5850
+	3300 5450 3300 5850
+Wire Wire Line
+	3250 5850 3300 5850
 $Comp
 L Connector:Conn_01x01_Female J2
@@
 Connect outer cable shield and plug shield to metal box.
 Text Notes 1800 6700 0    50   ~ 0
-For connection to the piezo crystals:\nUse shielded cable, with 4 leads.\nConnect outer cable shield to metal box. \nOuter end of cable shield may be connected to the outer box \nthat houses the crystals if that is used. If not, leave unconnected.
-Wire Wire Line
-	2400 5850 3200 5850
+For connection to the piezo crystals:\nUse shielded cable, with 3 leads.\nConnect outer cable shield to metal box. \nOuter end of cable shield may be connected to the outer box \nthat houses the crystals if that is used. If not, leave unconnected.
 $Comp
 L Connector:Conn_01x01_Female J9
 U 1 1 60AB3350
-P 3800 6050
-F 0 "J9" H 3828 6076 50  0000 L CNN
-F 1 "Conn_01x01_Female" H 3828 5985 50  0001 L CNN
-F 2 "MountingHole:MountingHole_2.2mm_M2_DIN965_Pad" H 3800 6050 50  0001 C CNN
-F 3 "~" H 3800 6050 50  0001 C CNN
-	1    3800 6050
+P 3250 6050
+F 0 "J9" H 3278 6076 50  0000 L CNN
+F 1 "Conn_01x01_Female" H 3278 5985 50  0001 L CNN
+F 2 "MountingHole:MountingHole_2.2mm_M2_DIN965_Pad" H 3250 6050 50  0001 C CNN
+F 3 "~" H 3250 6050 50  0001 C CNN
+	1    3250 6050
 	0    1    1    0
 $EndComp
@@
 L Connector:Conn_01x01_Female J8
 U 1 1 60AB34FC
-P 3200 6050
-F 0 "J8" H 3228 6076 50  0000 L CNN
-F 1 "Conn_01x01_Female" H 3228 5985 50  0001 L CNN
-F 2 "MountingHole:MountingHole_2.2mm_M2_DIN965_Pad" H 3200 6050 50  0001 C CNN
-F 3 "~" H 3200 6050 50  0001 C CNN
-	1    3200 6050
-	0    1    1    0
-$EndComp
-$Comp
-L Connector:Conn_01x01_Female J7
-U 1 1 60AB3506
-P 2050 6050
-F 0 "J7" H 2078 6076 50  0000 L CNN
-F 1 "Conn_01x01_Female" H 2078 5985 50  0001 L CNN
-F 2 "MountingHole:MountingHole_2.2mm_M2_DIN965_Pad" H 2050 6050 50  0001 C CNN
-F 3 "~" H 2050 6050 50  0001 C CNN
-	1    2050 6050
+P 2550 6050
+F 0 "J8" H 2578 6076 50  0000 L CNN
+F 1 "Conn_01x01_Female" H 2578 5985 50  0001 L CNN
+F 2 "MountingHole:MountingHole_2.2mm_M2_DIN965_Pad" H 2550 6050 50  0001 C CNN
+F 3 "~" H 2550 6050 50  0001 C CNN
+	1    2550 6050
 	0    1    1    0
 $EndComp
@@
 L Connector:Conn_01x01_Female J6
 U 1 1 60AB3510
-P 1450 6050
-F 0 "J6" H 1478 6076 50  0000 L CNN
-F 1 "Conn_01x01_Female" H 1478 5985 50  0001 L CNN
-F 2 "MountingHole:MountingHole_2.2mm_M2_DIN965_Pad" H 1450 6050 50  0001 C CNN
-F 3 "~" H 1450 6050 50  0001 C CNN
-	1    1450 6050
+P 1900 6050
+F 0 "J6" H 1928 6076 50  0000 L CNN
+F 1 "Conn_01x01_Female" H 1928 5985 50  0001 L CNN
+F 2 "MountingHole:MountingHole_2.2mm_M2_DIN965_Pad" H 1900 6050 50  0001 C CNN
+F 3 "~" H 1900 6050 50  0001 C CNN
+	1    1900 6050
 	0    1    1    0
 $EndComp
@@
 	5150 7450 850  7450
 Wire Notes Line
-	1550 5900 1700 5900
-Wire Notes Line
-	1700 5850 1700 5950
-Wire Notes Line
-	1750 5850 1750 5950
-Wire Notes Line
-	1750 5950 1800 5950
-Wire Notes Line
-	1800 5950 1800 5850
-Wire Notes Line
-	1800 5850 1750 5850
-Wire Notes Line
-	1850 5850 1850 5950
-Wire Notes Line
-	1850 5900 2000 5900
-Wire Notes Line
-	3300 5900 3450 5900
-Wire Notes Line
-	3450 5850 3450 5950
-Wire Notes Line
-	3500 5850 3500 5950
-Wire Notes Line
-	3500 5950 3550 5950
-Wire Notes Line
-	3550 5950 3550 5850
-Wire Notes Line
-	3550 5850 3500 5850
-Wire Notes Line
-	3600 5850 3600 5950
-Wire Notes Line
-	3600 5900 3750 5900
+	2000 5900 2150 5900
+Wire Notes Line
+	2150 5850 2150 5950
+Wire Notes Line
+	2200 5850 2200 5950
+Wire Notes Line
+	2200 5950 2250 5950
+Wire Notes Line
+	2250 5950 2250 5850
+Wire Notes Line
+	2250 5850 2200 5850
+Wire Notes Line
+	2300 5850 2300 5950
+Wire Notes Line
+	2300 5900 2450 5900
+Wire Notes Line
+	2750 5900 2900 5900
+Wire Notes Line
+	2900 5850 2900 5950
+Wire Notes Line
+	2950 5850 2950 5950
+Wire Notes Line
+	2950 5950 3000 5950
+Wire Notes Line
+	3000 5950 3000 5850
+Wire Notes Line
+	3000 5850 2950 5850
+Wire Notes Line
+	3050 5850 3050 5950
+Wire Notes Line
+	3050 5900 3200 5900
 Text Notes 2000 1000 0    50   ~ 0
 This line represent the outside of a metal box.
 Text Notes 7200 6800 0    50   ~ 0
-All resistors, FETs and capacitators are THT.\nUse film resistors and X7R caps!
-Text Notes 2200 5650 0    50   ~ 0
+All resistors, FETs and capacitators are THT.\nUse high tolerance film resistors and X7R caps!
+Text Notes 2050 5600 0    50   ~ 0
 2x 1N5230B-TR can be used.
 Text Notes 6000 4050 0    50   ~ 0
 Absolute Maximum Ratings@ 25 °C (unless otherwise stated)Maximum Temperatures\nStorage Temperature-65 to +150°C\nJunction Operating Temperature-55 to +150°C\nMaximum  Continuous Power Dissipation @ +25°C 400mW \nMaximum Currents:\nGate Forward CurrentIG(F)= 10mA\nMaximum Voltages:\nGate to SourceVGSS= 40\nVGate to DrainVGDS= 40V
-Text Notes 1600 6000 0    50   ~ 0
+Text Notes 2050 6000 0    50   ~ 0
 +
-Text Notes 3350 6000 0    50   ~ 0
+Text Notes 2800 6000 0    50   ~ 0
 +
 Text Notes 6050 4400 0    50   ~ 0
@@
 Wire Wire Line
 	4150 1500 4150 5150
+Wire Wire Line
+	2800 5750 2550 5750
+Wire Wire Line
+	2550 5750 2550 5850
+Connection ~ 1900 5450
+Wire Wire Line
+	1100 5450 1900 5450
+Connection ~ 3300 5450
 $EndSCHEMATC

Commit message: Add files via upload
Parts:
- removed J1: XLR3, Connector_PinSocket_2.54mm:PinSocket_1x03_P2.54mm_Vertical, symbol Connector:XLR3
- added J1, J10, J7: Conn_01x01_Female, MountingHole:MountingHole_2.2mm_M2_DIN965_Pad, symbol Connector:Conn_01x01_Female
Connections:
- net GND: now also J10.1 (Pin_1)
- net 2: now reaches C2.2, R1.2, R3.2
- net 2: now also J1.1 (Pin_1)
- net 3: now reaches R5.1, R7.2, R9.2
- net 3: now also J7.1 (Pin_1)
Other:
- note added: "*"
- note added: "If a 40 om resistor is not possible to get, replace Q1 \nwith a small jumper connected from pin 1 to 2 and use a 1K resistor in place of R12"
Changed lines of the file:
@@
 Wire Wire Line
 	2100 1500 2100 1900
-Wire Wire Line
-	2850 1500 4150 1500
-$Comp
-L Connector:XLR3 J1
-U 1 1 609DD8ED
-P 2550 1500
-F 0 "J1" H 2550 1865 50  0000 C CNN
-F 1 "XLR3" H 2550 1774 50  0000 C CNN
-F 2 "Connector_PinSocket_2.54mm:PinSocket_1x03_P2.54mm_Vertical" H 2550 1500 50  0001 C CNN
-F 3 " ~" H 2550 1500 50  0001 C CNN
-	1    2550 1500
-	-1   0    0    -1
-$EndComp
 Wire Notes Line
 	850  1000 5150 1000
@@
 	1100 5450 1900 5450
 Connection ~ 3300 5450
+$Comp
+L Connector:Conn_01x01_Female J10
+U 1 1 60BFB6E4
+P 2550 1300
+F 0 "J10" H 2578 1326 50  0000 L CNN
+F 1 "Conn_01x01_Female" H 2578 1235 50  0001 L CNN
+F 2 "MountingHole:MountingHole_2.2mm_M2_DIN965_Pad" H 2550 1300 50  0001 C CNN
+F 3 "~" H 2550 1300 50  0001 C CNN
+	1    2550 1300
+	0    -1   -1   0
+$EndComp
+$Comp
+L Connector:Conn_01x01_Female J7
+U 1 1 60BFB6EA
+P 2400 1300
+F 0 "J7" H 2428 1326 50  0000 L CNN
+F 1 "Conn_01x01_Female" H 2428 1235 50  0001 L CNN
+F 2 "MountingHole:MountingHole_2.2mm_M2_DIN965_Pad" H 2400 1300 50  0001 C CNN
+F 3 "~" H 2400 1300 50  0001 C CNN
+	1    2400 1300
+	0    -1   -1   0
+$EndComp
+$Comp
+L Connector:Conn_01x01_Female J1
+U 1 1 60BFB6F0
+P 2250 1300
+F 0 "J1" H 2278 1326 50  0000 L CNN
+F 1 "Conn_01x01_Female" H 2278 1235 50  0001 L CNN
+F 2 "MountingHole:MountingHole_2.2mm_M2_DIN965_Pad" H 2250 1300 50  0001 C CNN
+F 3 "~" H 2250 1300 50  0001 C CNN
+	1    2250 1300
+	0    -1   -1   0
+$EndComp
+Wire Wire Line
+	2550 1800 2400 1800
+Wire Wire Line
+	2400 1800 2400 1500
+Wire Wire Line
+	2550 1500 4150 1500
+Text Label 2100 1600 0    50   ~ 0
+2
+Text Label 2400 1600 0    50   ~ 0
+3
+Text Label 2600 1500 0    50   ~ 0
+1
+Text Notes 6000 4500 0    50   ~ 0
+If a 40 om resistor is not possible to get, replace Q1 \nwith a small jumper connected from pin 1 to 2 and use a 1K resistor in place of R12
+Text Notes 2500 4850 0    50   ~ 0
+*
 $EndSCHEMATC
